File: opamp_inverting_single.kicad_pcb (KiCad board)
At the start: 2 copper layers, 0 parts

Commit message: finished schematic and rough pcb layout
  updated libraries to get power nanofit
Parts:
- added C1: C, Capacitor_SMD:C_0805_2012Metric_Pad1.18x1.45mm_HandSolder, F.Cu at (154.0, 77.4)
- added C2: C, Capacitor_SMD:C_0805_2012Metric_Pad1.18x1.45mm_HandSolder, F.Cu at (163.0, 87.8)
- added C3: 0u1, Capacitor_SMD:C_0805_2012Metric_Pad1.18x1.45mm_HandSolder, F.Cu at (158.4, 93.5)
- added C4: 10u, Capacitor_SMD:C_0805_2012Metric_Pad1.18x1.45mm_HandSolder, B.Cu at (153.4, 90.7)
- added C5: 0u1, Capacitor_SMD:C_0805_2012Metric_Pad1.18x1.45mm_HandSolder, F.Cu at (153.5, 86.0)
- added C6: 10u, Capacitor_SMD:C_0805_2012Metric_Pad1.18x1.45mm_HandSolder, B.Cu at (153.5, 85.0)
- added C7: 0u1, Capacitor_SMD:C_0805_2012Metric_Pad1.18x1.45mm_HandSolder, F.Cu at (153.5, 90.8)
- added C8: 10u, Capacitor_SMD:C_0805_2012Metric_Pad1.18x1.45mm_HandSolder, B.Cu at (155.5, 87.8)
- added J1: Conn_Coaxial, Connector_Coaxial:SMA_Amphenol_132289_EdgeMount, F.Cu at (144.8, 75.9)
- added J2: Conn_Coaxial, Connector_Coaxial:SMA_Amphenol_132289_EdgeMount, F.Cu at (145.3, 98.4)
- added J3: Power-NanoFit-01x03, Connector_Molex:Molex_Nano-Fit_105313-xx03_1x03_P2.50mm_Horizontal, F.Cu at (150.8, 90.4)
- added R1: R_US, Resistor_SMD:R_0805_2012Metric_Pad1.20x1.40mm_HandSolder, F.Cu at (150.2, 78.2)
- added R2: R_US, Resistor_SMD:R_0805_2012Metric_Pad1.20x1.40mm_HandSolder, F.Cu at (158.3, 80.5)
- added R3: R_US, Resistor_SMD:R_0805_2012Metric_Pad1.20x1.40mm_HandSolder, F.Cu at (155.7, 82.0)
- added R4: R_US, Resistor_SMD:R_0805_2012Metric_Pad1.20x1.40mm_HandSolder, F.Cu at (161.0, 87.8)
- added R5: R_US, Resistor_SMD:R_0805_2012Metric_Pad1.20x1.40mm_HandSolder, F.Cu at (155.8, 93.5)
- added U1: LT1722xS8, Package_SO:SOIC-8_3.9x4.9mm_P1.27mm, F.Cu at (157.2, 87.9)

Commit message: some routing
Parts:
- added REF**: MountingHole_3.2mm_M3, MountingHole:MountingHole_3.2mm_M3, F.Cu at (160.8, 72.3)
- added REF**: MountingHole_3.2mm_M3, MountingHole:MountingHole_3.2mm_M3, F.Cu at (160.8, 102.3)
- moved J2 0.60 mm to (144.8, 98.8)
- moved J3 0.53 mm to (150.5, 90.0)
- moved C8 0.43 mm to (155.2, 87.5)
- moved R3 0.43 mm to (155.3, 81.7)
- moved C3 0.43 mm to (158.1, 93.3)
- moved C4 0.43 mm to (153.1, 90.5)
- moved C5 0.43 mm to (153.1, 85.7)
- moved C6 0.43 mm to (153.1, 84.7)
- moved R2 0.43 mm to (158.0, 80.2)
- moved U1 0.43 mm to (156.9, 87.6)
- moved C2 0.43 mm to (162.6, 87.5)
- moved C7 0.43 mm to (153.2, 90.5), turned to -90 degrees
- moved R4 0.43 mm to (160.6, 87.5)
- moved R5 0.43 mm to (155.5, 93.3)
- moved J1 0.11 mm to (144.8, 75.8)
Routing:
- net GND: track 0.00 -> 21.9 mm, vias 0 -> 7
- net /coax_out: track 0.00 -> 12.1 mm
- net +5V: track 0.00 -> 11.3 mm, vias 0 -> 2
- net /inv_in: track 0.00 -> 10.1 mm
- net /amp_out: track 0.00 -> 9.86 mm
- net -5V: track 0.00 -> 9.81 mm, vias 0 -> 1
- net /coax_in: track 0.00 -> 8.58 mm
- net /Cblock_Rin: track 0.00 -> 3.55 mm
- net /non_inv_in: track 0.00 -> 2.64 mm
Other:
- board outline added: 22.7 x 37 mm
- board text added: "2x M3 screw holes"

Commit message: Completed PCB
Routing:
- net GND: track 21.9 -> 24.1 mm
- net -5V: track 9.81 -> 11.2 mm, vias 1 -> 2
- added copper zone on In1.Cu, net +5V
- added copper zone on In2.Cu, net -5V
- added copper zone on B.Cu, net GND
Other:
- copper layers 2 -> 4
- board text added: "Inverting Single Opamp--SOIC8 HugonLabs v1.0 2022-04-28"
- board text removed: "2x M3 screw holes"
Changed lines of the file:
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@@
 (kicad_pcb (version 20211014) (generator pcbnew)
   (general
-    (thickness 1.6)
+    (thickness 4.69)
   )
   (paper "USLetter")
@@
     (title "Inverting Single Opamp -- SOIC8")
     (date "2022-04-28")
-    (rev "0.1")
+    (rev "1.0")
     (company "HugonLabs")
   )
   (layers
     (0 "F.Cu" signal)
+    (1 "In1.Cu" power)
+    (2 "In2.Cu" power)
     (31 "B.Cu" power)
     (32 "B.Adhes" user "B.Adhesive")
@@
       (layer "F.Cu" (type "copper") (thickness 0.035))
       (layer "dielectric 1" (type "core") (thickness 1.51) (material "FR4") (epsilon_r 4.5) (loss_tangent 0.02))
+      (layer "In1.Cu" (type "copper") (thickness 0.035))
+      (layer "dielectric 2" (type "prepreg") (thickness 1.51) (material "FR4") (epsilon_r 4.5) (loss_tangent 0.02))
+      (layer "In2.Cu" (type "copper") (thickness 0.035))
+      (layer "dielectric 3" (type "core") (thickness 1.51) (material "FR4") (epsilon_r 4.5) (loss_tangent 0.02))
       (layer "B.Cu" (type "copper") (thickness 0.035))
       (layer "B.Mask" (type "Bottom Solder Mask") (thickness 0.01))
@@
     (descr "Mounting Hole 3.2mm, no annular, M3")
     (tags "mounting hole 3.2mm no annular m3")
-    (attr exclude_from_pos_files exclude_from_bom)
+    (attr board_only exclude_from_pos_files exclude_from_bom)
     (fp_text reference "REF**" (at 0 -4.2) (layer "F.SilkS") hide
       (effects (font (size 1 1) (thickness 0.15)))
     )
-    (fp_text value "MountingHole_3.2mm_M3" (at 0 4.2) (layer "F.Fab")
-      (effects (font (size 1 1) (thickness 0.15)))
-    )
-    (fp_text user "${REFERENCE}" (at 0 0) (layer "F.Fab")
+    (fp_text value "MountingHole_3.2mm_M3" (at 15.1 -6.13) (layer "F.Fab")
+      (effects (font (size 1 1) (thickness 0.15)))
+    )
+    (fp_text user "${REFERENCE}" (at 0 0) (layer "F.Fab") hide
       (effects (font (size 1 1) (thickness 0.15)))
     )
@@
     (descr "Mounting Hole 3.2mm, no annular, M3")
     (tags "mounting hole 3.2mm no annular m3")
-    (attr exclude_from_pos_files exclude_from_bom)
+    (attr board_only exclude_from_pos_files exclude_from_bom)
     (fp_text reference "REF**" (at 0 -4.2) (layer "F.SilkS") hide
       (effects (font (size 1 1) (thickness 0.15)))
     )
-    (fp_text value "MountingHole_3.2mm_M3" (at 0 4.2) (layer "F.Fab")
-      (effects (font (size 1 1) (thickness 0.15)))
-    )
-    (fp_text user "${REFERENCE}" (at 0 0) (layer "F.Fab")
+    (fp_text value "MountingHole_3.2mm_M3" (at 14.24 5.81) (layer "F.Fab")
+      (effects (font (size 1 1) (thickness 0.15)))
+    )
+    (fp_text user "${REFERENCE}" (at 0 0) (layer "F.Fab") hide
       (effects (font (size 1 1) (thickness 0.15)))
     )
@@
   )
   (gr_rect locked (start 141.824989 68.799989) (end 164.525 105.799989) (layer "Edge.Cuts") (width 0.1) (fill none))
-  (gr_text "2x M3 screw holes" (at 173.324989 64.799989) (layer "Dwgs.User")
-    (effects (font (size 1 1) (thickness 0.15)))
+  (gr_text "Inverting Single\nOpamp--SOIC8\nHugonLabs\nv1.0 2022-04-28" (at 157.424989 79.639989 -45) (layer "B.SilkS")
+    (effects (font (size 1 1) (thickness 0.16)) (justify mirror))
+  )
+  (gr_text "Inverting Single\nOpamp--SOIC8\nHugonLabs\nv1.0\n2022-04-28" (at 152.834989 102.149989) (layer "F.SilkS")
+    (effects (font (size 0.6 0.6) (thickness 0.1)))
   )
   (dimension (type orthogonal) (layer "Dwgs.User")
@@
   (arc (start 152.024989 87.499989) (mid 152.336798 87.437966) (end 152.601137 87.26134) (width 0.2032) (layer "F.Cu") (net 1))
   (arc (start 147.904279 80.049989) (mid 147.969607 80.036994) (end 148.024989 79.999989) (width 0.2032) (layer "F.Cu") (net 1))
+  (segment (start 152.62603 88.95103) (end 153.099989 89.424989) (width 0.2032) (layer "B.Cu") (net 1))
   (segment (start 152.734564 86.790414) (end 152.024989 87.499989) (width 0.2032) (layer "B.Cu") (net 1))
   (arc (start 153.149989 85.787489) (mid 153.042024 86.330268) (end 152.734564 86.790414) (width 0.2032) (layer "B.Cu") (net 1))
+  (arc (start 152.024989 87.499989) (mid 152.181194 88.285287) (end 152.62603 88.95103) (width 0.2032) (layer "B.Cu") (net 1))
   (segment (start 152.050712 90.914266) (end 150.464989 89.999989) (width 0.2032) (layer "F.Cu") (net 2))
   (segment (start 158.074989 92.237489) (end 159.169812 92.237489) (width 0.2032) (layer "F.Cu") (net 2))
-  (segment (start 150.464989 89.999989) (end 151.216083 90.751083) (width 0.2032) (layer "F.Cu") (net 2))
   (segment (start 157.559989 90.074989) (end 157.559989 90.99417) (width 0.2032) (layer "F.Cu") (net 2))
   (segment (start 153.174989 91.562489) (end 152.050712 90.914266) (width 0.2032) (layer "F.Cu") (net 2))
@@
   (arc (start 159.169812 92.237489) (mid 159.186144 92.23424) (end 159.199989 92.224989) (width 0.2032) (layer "F.Cu") (net 2))
   (segment (start 154.590109 90.009868) (end 153.099989 91.499989) (width 0.2032) (layer "B.Cu") (net 2))
+  (segment (start 152.308653 91.172207) (end 152.050712 90.914266) (width 0.2032) (layer "B.Cu") (net 2))
+  (arc (start 153.099989 91.499989) (mid 152.671721 91.414801) (end 152.308653 91.172207) (width 0.2032) (layer "B.Cu") (net 2))
   (arc (start 155.199989 88.537489) (mid 155.041486 89.334335) (end 154.590109 90.009868) (width 0.2032) (layer "B.Cu") (net 2))
   (segment (start 151.977489 84.637489) (end 153.149989 84.637489) (width 0.2032) (layer "F.Cu") (net 3))
   (segment (start 151.340141 84.637489) (end 151.977489 84.637489) (width 0.2032) (layer "F.Cu") (net 3))
+  (segment (start 153.174989 89.487489) (end 153.554989 89.487489) (width 0.2032) (layer "F.Cu") (net 3))
+  (segment (start 153.554989 89.487489) (end 153.554989 88.431589) (width 0.2032) (layer "F.Cu") (net 3))
   (segment (start 153.149989 84.637489) (end 153.84306 84.637489) (width 0.2032) (layer "F.Cu") (net 3))
   (via (at 151.977489 84.637489) (size 0.508) (drill 0.254) (layers "F.Cu" "B.Cu") (net 3))
+  (via (at 153.554989 88.431589) (size 0.508) (drill 0.254) (layers "F.Cu" "B.Cu") (net 3))
   (arc (start 153.84306 84.637489) (mid 154.480009 84.764186) (end 155.019989 85.124989) (width 0.2032) (layer "F.Cu") (net 3))
   (arc (start 150.464989 84.999989) (mid 150.866512 84.7317) (end 151.340141 84.637489) (width 0.2032) (layer "F.Cu") (net 3))
@@
   (segment (start 156.289989 85.124989) (end 156.289989 85.054705) (width 0.2032) (layer "F.Cu") (net 12))
   (arc (start 156.289989 85.054705) (mid 156.039194 83.793872) (end 155.324989 82.724989) (width 0.2032) (layer "F.Cu") (net 12))
+  (zone (net 2) (net_name "+5V") (layer "In1.Cu") (hatch edge 0.508)
+    (connect_pads (clearance 0.508))
+    (min_thickness 0.254) (filled_areas_thickness no)
+    (fill yes (thermal_gap 0.508) (thermal_bridge_width 0.508))
+    (polygon
+      (pts
+        (xy 156.824989 74.799989)
+        (xy 158.324989 76.299989)
+        (xy 163.824989 76.299989)
+        (xy 163.824989 98.299989)
+        (xy 158.324989 98.299989)
+        (xy 156.824989 99.799989)
+        (xy 156.824989 105.299989)
+        (xy 142.324989 105.299989)
+        (xy 142.324989 69.299989)
+        (xy 156.824989 69.299989)
+      )
+    )
+  )
+  (zone (net 3) (net_name "-5V") (layer "In2.Cu") (hatch edge 0.508)
+    (connect_pads (clearance 0.508))
+    (min_thickness 0.254) (filled_areas_thickness no)
+    (fill yes (thermal_gap 0.508) (thermal_bridge_width 0.508))
+    (polygon
+      (pts
+        (xy 156.824989 74.799989)
+        (xy 158.324989 76.299989)
+        (xy 163.824989 76.299989)
+        (xy 163.824989 98.299989)
+        (xy 158.324989 98.299989)
+        (xy 156.824989 99.799989)
+        (xy 156.824989 105.299989)
+        (xy 142.324989 105.299989)
+        (xy 142.324989 69.299989)
+        (xy 156.824989 69.299989)
+      )
+    )
+  )
+  (zone (net 0) (net_name "") (layers "In1.Cu" "In2.Cu" "B.Cu") (name "Inverting input fill exclusion") (hatch edge 0.508)
+    (connect_pads (clearance 0))
+    (min_thickness 0.254)
+    (keepout (tracks not_allowed) (vias not_allowed) (pads not_allowed ) (copperpour not_allowed) (footprints not_allowed))
+    (fill (thermal_gap 0.508) (thermal_bridge_width 0.508))
+    (polygon
+      (pts
+        (xy 159.024989 80.499989)
+        (xy 159.024989 81.999989)
+        (xy 157.924989 82.099989)
+        (xy 157.924989 83.699989)
+        (xy 158.124989 83.999989)
+        (xy 158.224989 85.299989)
+        (xy 158.224989 86.199989)
+        (xy 159.324989 86.199989)
+        (xy 159.924989 85.699989)
+        (xy 163.424989 85.599989)
+        (xy 163.624989 85.799989)
+        (xy 163.624989 87.199989)
+        (xy 163.324989 87.299989)
+        (xy 159.824989 87.399989)
+        (xy 159.324989 86.899989)
+        (xy 157.924989 86.799989)
+        (xy 157.524989 86.399989)
+        (xy 157.024989 86.199989)
+        (xy 156.924989 80.399989)
+        (xy 157.024989 80.299989)
+        (xy 158.724989 80.299989)
+      )
+    )
+  )
+  (zone (net 1) (net_name "GND") (layer "B.Cu") (hatch edge 0.508)
+    (connect_pads (clearance 0.508))
+    (min_thickness 0.254) (filled_areas_thickness no)
+    (fill yes (thermal_gap 0.508) (thermal_bridge_width 0.508))
+    (polygon
+      (pts
+        (xy 156.824989 74.799989)
+        (xy 158.324989 76.299989)
+        (xy 163.824989 76.299989)
+        (xy 163.824989 98.299989)
+        (xy 158.324989 98.299989)
+        (xy 156.824989 99.799989)
+        (xy 156.824989 105.299989)
+        (xy 142.324989 105.299989)
+        (xy 142.324989 69.299989)
+        (xy 156.824989 69.299989)
+      )
+    )
+  )
 )
