File: opamp_inverting_single.kicad_sch (KiCad schematic)
At the start: 0 parts

Commit message: finished schematic and rough pcb layout
  updated libraries to get power nanofit
Parts:
- added C1, C2, C3, C4, C5, C6, C7, C8: (no value), symbol Device:C
- added J1, J2: (no value), symbol Connector:Conn_Coaxial
- added J3: (no value), symbol HugonLib:Power-NanoFit-01x03
- added R1, R2, R3, R4, R5: (no value), symbol Device:R_US
- added U1: (no value), symbol HugonLib:LT1722xS8
Connections:
- new net +5V: C3.2, C4.2, C7.2, C8.2, J3.1 (Pin_1), U1.7 (V+)
- new net -5V: C5.1, C6.1, C7.1, C8.1, J3.3 (Pin_3), U1.4 (V-)
- new net Cblock_Rin: C1.2, R2.1
- new net GND: C3.1, C4.1, C5.2, C6.2, J1.2 (Ext), J2.2 (Ext), J3.2 (Pin_2), R1.1, R3.2
- new net amp_out: C2.2, R4.2, R5.1, U1.6 (Out)
- new net coax_in: C1.1, J1.1 (In), R1.2
- new net coax_out: J2.1 (In), R5.2
- new net inv_in: C2.1, R2.2, R4.1, U1.2 (-in)
- new net non_inv_in: R3.1, U1.3 (+in)

Commit message: Completed PCB
Parts:
- C1, C2: value (none) -> C; footprint (none) -> Capacitor_SMD:C_0805_2012Metric_Pad1.18x1.45mm_HandSolder
- C3, C5, C7: value (none) -> 0u1; footprint (none) -> Capacitor_SMD:C_0805_2012Metric_Pad1.18x1.45mm_HandSolder
- C4, C6, C8: value (none) -> 10u; footprint (none) -> Capacitor_SMD:C_0805_2012Metric_Pad1.18x1.45mm_HandSolder
- J1, J2: value (none) -> Conn_Coaxial; footprint (none) -> Connector_Coaxial:SMA_Amphenol_132289_EdgeMount
- J3: value (none) -> Power-NanoFit-01x03; footprint (none) -> Connector_Molex:Molex_Nano-Fit_105313-xx03_1x03_P2.50mm_Horizontal
- R1, R2, R3, R4, R5: value (none) -> R_US; footprint (none) -> Resistor_SMD:R_0805_2012Metric_Pad1.20x1.40mm_HandSolder
- U1: value (none) -> LT1722xS8; footprint (none) -> Package_SO:SOIC-8_3.9x4.9mm_P1.27mm
Changed lines of the file:
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@@
     (title "Inverting Single Opamp -- SOIC8")
     (date "2022-04-28")
-    (rev "0.1")
+    (rev "1.0")
     (company "HugonLabs")
   )
@@
     (in_bom yes) (on_board yes) (fields_autoplaced)
     (property "Reference" "C2" (id 0) (at 146.05 46.99 90))
-    (property "Value" "" (id 1) (at 146.05 49.53 90))
-    (property "Footprint" "" (id 2) (at 149.86 53.6448 0)
+    (property "Value" "C" (id 1) (at 146.05 49.53 90))
+    (property "Footprint" "Capacitor_SMD:C_0805_2012Metric_Pad1.18x1.45mm_HandSolder" (id 2) (at 149.86 53.6448 0)
       (effects (font (size 1.27 1.27)) hide)
     )
@@
       (effects (font (size 1.27 1.27)) (justify right))
     )
-    (property "Value" "" (id 1) (at 104.14 102.8699 0)
-      (effects (font (size 1.27 1.27)) (justify right))
-    )
-    (property "Footprint" "" (id 2) (at 100.584 101.346 90)
+    (property "Value" "R_US" (id 1) (at 104.14 102.8699 0)
+      (effects (font (size 1.27 1.27)) (justify right))
+    )
+    (property "Footprint" "Resistor_SMD:R_0805_2012Metric_Pad1.20x1.40mm_HandSolder" (id 2) (at 100.584 101.346 90)
       (effects (font (size 1.27 1.27)) hide)
     )
@@
       (effects (font (size 1.27 1.27)) (justify left))
     )
-    (property "Value" "" (id 1) (at 134.62 109.2199 0)
+    (property "Value" "R_US" (id 1) (at 134.62 109.2199 0)
       (effects (font (size 1.27 1.27)) (justify left))
     )
-    (property "Footprint" "" (id 2) (at 133.096 108.204 90)
+    (property "Footprint" "Resistor_SMD:R_0805_2012Metric_Pad1.20x1.40mm_HandSolder" (id 2) (at 133.096 108.204 90)
       (effects (font (size 1.27 1.27)) hide)
     )
@@
     (in_bom yes) (on_board yes) (fields_autoplaced)
     (property "Reference" "R2" (id 0) (at 124.46 86.36 90))
-    (property "Value" "" (id 1) (at 124.46 88.9 90))
-    (property "Footprint" "" (id 2) (at 124.714 91.694 90)
+    (property "Value" "R_US" (id 1) (at 124.46 88.9 90))
+    (property "Footprint" "Resistor_SMD:R_0805_2012Metric_Pad1.20x1.40mm_HandSolder" (id 2) (at 124.714 91.694 90)
       (effects (font (size 1.27 1.27)) hide)
     )
@@
       (effects (font (size 1.27 1.27)) (justify left))
     )
-    (property "Value" "" (id 1) (at 78.74 156.21 90)
+    (property "Value" "Power-NanoFit-01x03" (id 1) (at 78.74 156.21 90)
       (effects (font (size 1.27 1.27)) (justify left))
     )
-    (property "Footprint" "" (id 2) (at 96.52 151.13 0)
+    (property "Footprint" "Connector_Molex:Molex_Nano-Fit_105313-xx03_1x03_P2.50mm_Horizontal" (id 2) (at 96.52 151.13 0)
       (effects (font (size 1.27 1.27)) hide)
     )
@@
       (effects (font (size 1.27 1.27)) (justify right))
     )
-    (property "Value" "" (id 1) (at 233.68 146.0499 0)
-      (effects (font (size 1.27 1.27)) (justify right))
-    )
-    (property "Footprint" "" (id 2) (at 228.9048 140.97 0)
+    (property "Value" "10u" (id 1) (at 233.68 146.0499 0)
+      (effects (font (size 1.27 1.27)) (justify right))
+    )
+    (property "Footprint" "Capacitor_SMD:C_0805_2012Metric_Pad1.18x1.45mm_HandSolder" (id 2) (at 228.9048 140.97 0)
       (effects (font (size 1.27 1.27)) hide)
     )
@@
       (effects (font (size 1.27 1.27)) (justify right))
     )
-    (property "Value" "" (id 1) (at 219.71 146.0499 0)
-      (effects (font (size 1.27 1.27)) (justify right))
-    )
-    (property "Footprint" "" (id 2) (at 214.9348 140.97 0)
+    (property "Value" "0u1" (id 1) (at 219.71 146.0499 0)
+      (effects (font (size 1.27 1.27)) (justify right))
+    )
+    (property "Footprint" "Capacitor_SMD:C_0805_2012Metric_Pad1.18x1.45mm_HandSolder" (id 2) (at 214.9348 140.97 0)
       (effects (font (size 1.27 1.27)) hide)
     )
@@
     (in_bom yes) (on_board yes) (fields_autoplaced)
     (property "Reference" "R5" (id 0) (at 177.8 90.17 90))
-    (property "Value" "" (id 1) (at 177.8 92.71 90))
-    (property "Footprint" "" (id 2) (at 178.054 95.504 90)
+    (property "Value" "R_US" (id 1) (at 177.8 92.71 90))
+    (property "Footprint" "Resistor_SMD:R_0805_2012Metric_Pad1.20x1.40mm_HandSolder" (id 2) (at 178.054 95.504 90)
       (effects (font (size 1.27 1.27)) hide)
     )
@@
       (effects (font (size 1.27 1.27)) (justify right))
     )
-    (property "Value" "" (id 1) (at 193.04 146.0499 0)
-      (effects (font (size 1.27 1.27)) (justify right))
-    )
-    (property "Footprint" "" (id 2) (at 188.2648 140.97 0)
+    (property "Value" "0u1" (id 1) (at 193.04 146.0499 0)
+      (effects (font (size 1.27 1.27)) (justify right))
+    )
+    (property "Footprint" "Capacitor_SMD:C_0805_2012Metric_Pad1.18x1.45mm_HandSolder" (id 2) (at 188.2648 140.97 0)
       (effects (font (size 1.27 1.27)) hide)
     )
@@
       (effects (font (size 1.27 1.27)) (justify right))
     )
-    (property "Value" "" (id 1) (at 166.37 146.0499 0)
-      (effects (font (size 1.27 1.27)) (justify right))
-    )
-    (property "Footprint" "" (id 2) (at 161.5948 140.97 0)
+    (property "Value" "0u1" (id 1) (at 166.37 146.0499 0)
+      (effects (font (size 1.27 1.27)) (justify right))
+    )
+    (property "Footprint" "Capacitor_SMD:C_0805_2012Metric_Pad1.18x1.45mm_HandSolder" (id 2) (at 161.5948 140.97 0)
       (effects (font (size 1.27 1.27)) hide)
     )
@@
       (effects (font (size 1.27 1.27)) (justify left))
     )
-    (property "Value" "" (id 1) (at 200.66 98.0831 0)
+    (property "Value" "Conn_Coaxial" (id 1) (at 200.66 98.0831 0)
       (effects (font (size 1.27 1.27)) (justify left))
     )
-    (property "Footprint" "" (id 2) (at 198.12 96.52 0)
+    (property "Footprint" "Connector_Coaxial:SMA_Amphenol_132289_EdgeMount" (id 2) (at 198.12 96.52 0)
       (effects (font (size 1.27 1.27)) hide)
     )
@@
     (in_bom yes) (on_board yes)
     (property "Reference" "U1" (id 0) (at 156.21 86.36 0))
-    (property "Value" "" (id 1) (at 156.21 88.9 0))
-    (property "Footprint" "" (id 2) (at 138.43 116.84 0)
+    (property "Value" "LT1722xS8" (id 1) (at 156.21 88.9 0))
+    (property "Footprint" "Package_SO:SOIC-8_3.9x4.9mm_P1.27mm" (id 2) (at 138.43 116.84 0)
       (effects (font (size 1.27 1.27)) hide)
     )
@@
     (in_bom yes) (on_board yes) (fields_autoplaced)
     (property "Reference" "C1" (id 0) (at 111.76 85.09 90))
-    (property "Value" "" (id 1) (at 111.76 87.63 90))
-    (property "Footprint" "" (id 2) (at 115.57 91.7448 0)
+    (property "Value" "C" (id 1) (at 111.76 87.63 90))
+    (property "Footprint" "Capacitor_SMD:C_0805_2012Metric_Pad1.18x1.45mm_HandSolder" (id 2) (at 115.57 91.7448 0)
       (effects (font (size 1.27 1.27)) hide)
     )
@@
     (in_bom yes) (on_board yes) (fields_autoplaced)
     (property "Reference" "J1" (id 0) (at 89.2174 85.09 0))
-    (property "Value" "" (id 1) (at 89.2174 87.63 0))
-    (property "Footprint" "" (id 2) (at 88.9 92.71 0)
+    (property "Value" "Conn_Coaxial" (id 1) (at 89.2174 87.63 0))
+    (property "Footprint" "Connector_Coaxial:SMA_Amphenol_132289_EdgeMount" (id 2) (at 88.9 92.71 0)
       (effects (font (size 1.27 1.27)) hide)
     )
@@
       (effects (font (size 1.27 1.27)) (justify right))
     )
-    (property "Value" "" (id 1) (at 180.34 146.0499 0)
-      (effects (font (size 1.27 1.27)) (justify right))
-    )
-    (property "Footprint" "" (id 2) (at 175.5648 140.97 0)
+    (property "Value" "10u" (id 1) (at 180.34 146.0499 0)
+      (effects (font (size 1.27 1.27)) (justify right))
+    )
+    (property "Footprint" "Capacitor_SMD:C_0805_2012Metric_Pad1.18x1.45mm_HandSolder" (id 2) (at 175.5648 140.97 0)
       (effects (font (size 1.27 1.27)) hide)
     )
@@
       (effects (font (size 1.27 1.27)) (justify right))
     )
-    (property "Value" "" (id 1) (at 205.74 146.0499 0)
-      (effects (font (size 1.27 1.27)) (justify right))
-    )
-    (property "Footprint" "" (id 2) (at 200.9648 140.97 0)
+    (property "Value" "10u" (id 1) (at 205.74 146.0499 0)
+      (effects (font (size 1.27 1.27)) (justify right))
+    )
+    (property "Footprint" "Capacitor_SMD:C_0805_2012Metric_Pad1.18x1.45mm_HandSolder" (id 2) (at 200.9648 140.97 0)
       (effects (font (size 1.27 1.27)) hide)
     )
@@
     (in_bom yes) (on_board yes) (fields_autoplaced)
     (property "Reference" "R4" (id 0) (at 146.05 64.77 90))
-    (property "Value" "" (id 1) (at 146.05 67.31 90))
-    (property "Footprint" "" (id 2) (at 146.304 70.104 90)
-      (effects (font (size 1.27 1.27)) hide)
-    )
+    (property "Value" "R_US" (id 1) (at 146.05 67.31 90))
+    (property "Footprint" "Resistor_SMD:R_0805_2012Metric_Pad1.20x1.40mm_HandSolder" (id 2) (at 146.304 70.104 90)
+      (effects (font (size 1.27 1.27)) hide)
+    )
